File: KiCad/Main Board/Electronic Target V3.sch (KiCad schematic (older format))
At the start: 69 parts, among them IC1 FT230XS-U, J1 Conn_02x06_Odd_Even, J2 Conn_02x04_Odd_Even, J3 Conn_01x06, J4 MINI USB, J5 Conn_01x04, Q1 CSD13383F4, Q2 CSD1338F4, U1 LM75AIMX_NOPB, U2 74LV8154, U3 LM339, U4 74HC74, U5 74HC00, U6 74LV8154, U7 74HC74, U8 NMA0505SC, X1 8M0

Commit message: Priming Version 3.0
Version 3.0 is the new board which supports LED lighting and other features.
Parts:
- removed J3: Conn_01x06, symbol Connector_Generic:Conn_01x06
- removed J4: MINI USB, symbol Connector_Generic:Conn_01x05
- removed J5: Conn_01x04, symbol Connector_Generic:Conn_01x04
- removed Q1: CSD13383F4, symbol Device:Q_NMOS_DGS
- removed Q2: CSD1338F4, symbol Device:Q_NMOS_DGS
- removed R18, R19: 0R, symbol Device:R
- added J3: MINI USB, symbol Connector_Generic:Conn_01x05
- added J6: Conn_01x06, symbol Connector_Generic:Conn_01x06
- C13: value 47pF -> 100nF
- C14: value 100nF -> 47pF
- C15: value 47pF -> 4k7
- C16: value 4u7F -> 47pF
- R11: value 2K0 -> 4K7
- R15: value 10K0 -> 10k0
Connections:
- net labels added: SPARE
- net labels removed: SPARE_1, SPARE_2
- wire segments 453 -> 428
Other:
- note added: "Copyright 2020 ten-point-nine\n\nPermission is hereby granted, free of charge, to any person obtaining a copy \nof this software and associated documentation files (the "Software"), to deal\nin the Software without restriction, including without limitation the rights to \nuse, copy, modify, merge, publish, distribute, sublicense, and/or sell copies \nof the Software, and to permit persons to whom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"
- note removed: "AUX\nPORT"
- note removed: "CHANGED"
- note removed: "Copyright 2020-2021 ten-point-nine\n\nPermission is hereby granted, free of charge, to any person obtaining a copy \nof this software and associated documentation files (the “Software”), to deal\nin the Software without restriction, including without limitation the rights to \nuse, copy, modify, merge, publish, distribute, sublicense, and/or sell copies \nof the Software, and to permit persons to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"
- note removed: "LED\nDRIVE"
- note removed: "NEW"
- note removed: "POPULATE R19 ONLY"
- note removed: "Value Changed"
- moved on the sheet: C11, U3E, V-5
